Commit message: hand-e gripper

File: drims2_description/urdf/ur5e/ur5e_cell.urdf.xacro (robot description, xacro)
@@ -64,4 +64,13 @@
          </material>
       </visual>
+      <collision>
+         <geometry>
+            <box size="${table_length} ${table_width} ${table_thickness}"/>
+         </geometry>
+         <origin xyz="0 0 -${table_thickness/2}" rpy="0 0 0"/>
+         <material name="brown">
+            <color rgba="0.4 0.2 0 1"/>
+         </material>
+      </collision>
    </link>
    <joint name="world_to_table" type="fixed">
@@ -74,11 +83,20 @@
          <visual>
             <geometry>
-            <box size="${leg_width} ${leg_width} ${z}"/>
+               <box size="${leg_width} ${leg_width} ${z}"/>
             </geometry>
             <origin xyz="0 0 ${z / 2}" rpy="0 0 0"/>
             <material name="black">
-            <color rgba="0.1 0.1 0.1 1"/>
+               <color rgba="0.1 0.1 0.1 1"/>
             </material>
          </visual>
+         <collision>
+            <geometry>
+               <box size="${leg_width} ${leg_width} ${z}"/>
+            </geometry>
+            <origin xyz="0 0 ${z / 2}" rpy="0 0 0"/>
+            <material name="black">
+               <color rgba="0.1 0.1 0.1 1"/>
+            </material>
+      </collision>
       </link>
       <joint name="joint_${name}" type="fixed">
@@ -101,5 +119,5 @@
          <origin xyz="${xyz}" rpy="0 0 0"/>
          <material name="red_transparent">
-         <color rgba="1.0 0.0 0.0 0.3"/>
+         <color rgba="1.0 1.0 0.5 0.3"/>
          </material>
       </visual>
@@ -173,11 +191,26 @@
       <origin xyz="${-table_length/2.0 + 0.1} 0 0" rpy="0 0 0"/>
    </xacro:ur_robot>
-    <!-- Robotiq 2f-140 gripper -->
-    <xacro:arg name="com_port" default="/dev/ttyUSB0" />
-    <!-- Import macros -->
-    <xacro:include filename="$(find robotiq_description)/urdf/robotiq_2f_140_macro.urdf.xacro" />
+    <!-- Robotiq Hand-e gripper -->
+   <xacro:arg name="com_port" default="/dev/ttyUSB0" />
+   <xacro:include filename="$(find robotiq_hande_description)/urdf/robotiq_hande_gripper.xacro" />
+   <xacro:robotiq_hande_gripper
+     name="robotiq_hande_gripper"
+     prefix=""
+     parent="tool0"
+     grip_pos_min="0.0"
+     grip_pos_max="0.025"
+     tty="$(arg com_port)"
+     baudrate="115200"
+     parity="N"
+     data_bits="8"
+     stop_bit="1"
+     slave_id="9"
+     use_fake_hardware="$(arg use_fake_hardware)"
+   />
+   <!-- Robotiq 2f-140 gripper -->
+    <!-- <xacro:include filename="$(find robotiq_description)/urdf/robotiq_hande_gripper.urdf.xacro" />
     <xacro:robotiq_gripper name="RobotiqGripperHardwareInterface" prefix="" parent="tool0" use_fake_hardware="$(arg use_fake_hardware)" com_port="$(arg com_port)">
         <origin xyz="0 0 0" rpy="0 0 0" />
-    </xacro:robotiq_gripper>
+    </xacro:robotiq_gripper> -->
    <link name="tip"/>
    <joint name="tool0_to_tip" type="fixed">

File: drims2_description/urdf/yumi/yumi_cell.urdf.xacro (robot description, xacro)
@@ -19,4 +19,13 @@
          </material>
       </visual>
+      <collision>
+         <geometry>
+            <box size="${table_length} ${table_width} ${table_thickness}"/>
+         </geometry>
+         <origin xyz="0 0 -${table_thickness/2}" rpy="0 0 0"/>
+         <material name="brown">
+            <color rgba="0.4 0.2 0 1"/>
+         </material>
+      </collision>
    </link>
    <joint name="world_to_table" type="fixed">
@@ -29,11 +38,20 @@
          <visual>
             <geometry>
-            <box size="${leg_width} ${leg_width} ${z}"/>
+               <box size="${leg_width} ${leg_width} ${z}"/>
             </geometry>
             <origin xyz="0 0 ${z / 2}" rpy="0 0 0"/>
             <material name="black">
-            <color rgba="0.1 0.1 0.1 1"/>
+               <color rgba="0.1 0.1 0.1 1"/>
             </material>
          </visual>
+         <collision>
+            <geometry>
+               <box size="${leg_width} ${leg_width} ${z}"/>
+            </geometry>
+            <origin xyz="0 0 ${z / 2}" rpy="0 0 0"/>
+            <material name="black">
+               <color rgba="0.1 0.1 0.1 1"/>
+            </material>
+      </collision>
       </link>
       <joint name="joint_${name}" type="fixed">
@@ -56,5 +74,5 @@
          <origin xyz="${xyz}" rpy="0 0 0"/>
          <material name="red_transparent">
-         <color rgba="1.0 0.0 0.0 0.3"/>
+         <color rgba="1.0 1.0 0.5 0.3"/>
          </material>
       </visual>

Commit message: minor fix

File: drims2_description/urdf/ur5e/ur5e_cell.urdf.xacro (robot description, xacro)
@@ -217,5 +217,5 @@
       <parent link="tool0"/>
       <child link="tip"/>
-      <origin xyz="0 0 0.2" rpy="0 0 0"/>
+      <origin xyz="0 0 0.15" rpy="0 0 0"/>
    </joint>
 </robot>

Commit message: Real UR setup

File: drims2_description/urdf/ur5e/ur5e_cell.urdf.xacro (robot description, xacro)
@@ -18,7 +18,7 @@
    <!-- ros2_control related parameters -->
    <xacro:arg name="headless_mode" default="false" />
-   <xacro:arg name="script_filename" default=""/>
-   <xacro:arg name="output_recipe_filename" default=""/>
-   <xacro:arg name="input_recipe_filename" default=""/>
+   <xacro:arg name="script_filename" default="$(find ur_client_library)/resources/external_control.urscript"/>
+   <xacro:arg name="input_recipe_filename" default="$(find ur_robot_driver)/resources/rtde_input_recipe.txt"/>
+   <xacro:arg name="output_recipe_filename" default="$(find ur_robot_driver)/resources/rtde_output_recipe.txt"/>
    <xacro:arg name="reverse_ip" default="0.0.0.0"/>
    <xacro:arg name="script_command_port" default="50004"/>
@@ -27,6 +27,6 @@
    <xacro:arg name="trajectory_port" default="50003"/>
    <!--   tool communication related parameters-->
-   <xacro:arg name="use_tool_communication" default="false" />
-   <xacro:arg name="tool_voltage" default="0" />
+   <xacro:arg name="use_tool_communication" default="true" />
+   <xacro:arg name="tool_voltage" default="24" />
    <xacro:arg name="tool_parity" default="0" />
    <xacro:arg name="tool_baud_rate" default="115200" />
@@ -192,5 +192,5 @@
    </xacro:ur_robot>
     <!-- Robotiq Hand-e gripper -->
-   <xacro:arg name="com_port" default="/dev/ttyUSB0" />
+   <xacro:arg name="com_port" default="/tmp/ttyUR" />
    <xacro:include filename="$(find robotiq_hande_description)/urdf/robotiq_hande_gripper.xacro" />
    <xacro:robotiq_hande_gripper
@@ -206,6 +206,17 @@
      stop_bit="1"
      slave_id="9"
-     use_fake_hardware="$(arg use_fake_hardware)"
+     use_fake_hardware="true"
    />
+   <!-- <xacro:include filename="$(find robotiq_description)/urdf/robotiq_hand_e_macro.urdf.xacro"/>
+   <xacro:include filename="$(find robotiq_description)/urdf/hand_e.ros2_control.xacro"/>
+   <xacro:robotiq_hande prefix="" parent="tool0" >
+      <origin xyz="0 0 0" rpy="0 0 0" />
+   </xacro:robotiq_hande>
+   <xacro:robotiq_hande_ros2_control
+      name="robotiq_hande"
+      prefix=""
+      use_mock_hardware="$(arg use_fake_hardware)"
+      com_port="$(arg com_port)"
+      /> -->
    <!-- Robotiq 2f-140 gripper -->
     <!-- <xacro:include filename="$(find robotiq_description)/urdf/robotiq_hande_gripper.urdf.xacro" />

Commit message: fixes

File: drims2_description/urdf/ur5e/ur5e_cell.urdf.xacro (robot description, xacro)
@@ -192,5 +192,4 @@
    </xacro:ur_robot>
     <!-- Robotiq Hand-e gripper -->
-   <xacro:arg name="com_port" default="/tmp/ttyUR" />
    <xacro:include filename="$(find robotiq_hande_description)/urdf/robotiq_hande_gripper.xacro" />
    <xacro:robotiq_hande_gripper
@@ -200,5 +199,5 @@
      grip_pos_min="0.0"
      grip_pos_max="0.025"
-     tty="$(arg com_port)"
+     tty="/tmp/ttyUR"
      baudrate="115200"
      parity="N"
@@ -206,22 +205,6 @@
      stop_bit="1"
      slave_id="9"
-     use_fake_hardware="true"
+     use_fake_hardware="$(arg use_fake_hardware)"
    />
-   <!-- <xacro:include filename="$(find robotiq_description)/urdf/robotiq_hand_e_macro.urdf.xacro"/>
-   <xacro:include filename="$(find robotiq_description)/urdf/hand_e.ros2_control.xacro"/>
-   <xacro:robotiq_hande prefix="" parent="tool0" >
-      <origin xyz="0 0 0" rpy="0 0 0" />
-   </xacro:robotiq_hande>
-   <xacro:robotiq_hande_ros2_control
-      name="robotiq_hande"
-      prefix=""
-      use_mock_hardware="$(arg use_fake_hardware)"
-      com_port="$(arg com_port)"
-      /> -->
-   <!-- Robotiq 2f-140 gripper -->
-    <!-- <xacro:include filename="$(find robotiq_description)/urdf/robotiq_hande_gripper.urdf.xacro" />
-    <xacro:robotiq_gripper name="RobotiqGripperHardwareInterface" prefix="" parent="tool0" use_fake_hardware="$(arg use_fake_hardware)" com_port="$(arg com_port)">
-        <origin xyz="0 0 0" rpy="0 0 0" />
-    </xacro:robotiq_gripper> -->
    <link name="tip"/>
    <joint name="tool0_to_tip" type="fixed">
