Commit message: First try

File: drims2_description/urdf/ur5e_2fg7/ur5e_2fg7_cell.urdf.xacro (robot description, xacro)
@@ -179,5 +179,5 @@
    <xacro:onrobot_2fg7_gripper
       parent="tool0"
-      prefix="2fg7_gripper_"
+      prefix=""
    />
    <link name="tip"/>
@@ -187,6 +187,32 @@
       <origin xyz="0 0 0.15" rpy="0 0 0"/>
    </joint>
-   <!-- ros2_control fake system for gripper -->
+   <!-- Replace the fake hardware section with this: -->
+   <xacro:unless value="$(arg use_fake_hardware)">
+   <ros2_control name="onrobot_2fg7_gripper" type="system">
+      <hardware>
+         <plugin>onrobot_driver/OnRobotGripperHardwareInterface</plugin>
+         <param name="ip_address">192.168.1.1</param>
+         <param name="port">502</param>
+         <param name="gripper_type">2FG7</param>
+         <param name="max_width">0.085</param>
+         <param name="min_width">0.0</param>
+         <param name="max_force">100.0</param>
+      </hardware>
+      <joint name="left_finger_joint">
+         <command_interface name="position"/>
+         <state_interface name="position"/>
+         <state_interface name="velocity"/>
+         <state_interface name="effort"/>
+      </joint>
+      <joint name="right_finger_joint">
+         <command_interface name="position"/>
+         <state_interface name="position"/>
+         <state_interface name="velocity"/>
+         <state_interface name="effort"/>
+      </joint>
+   </ros2_control>
+   </xacro:unless>
    <xacro:if value="$(arg use_fake_hardware)">
+   <!-- Keep the fake hardware for simulation -->
    <ros2_control name="onrobot_2fg7_gripper" type="system">
       <hardware>
@@ -205,4 +231,4 @@
       </joint>
    </ros2_control>
-   </xacro:if>
+</xacro:if>
 </robot>

Commit message: Second try

File: drims2_description/urdf/ur5e_2fg7/ur5e_2fg7_cell.urdf.xacro (robot description, xacro)
@@ -187,6 +187,26 @@
       <origin xyz="0 0 0.15" rpy="0 0 0"/>
    </joint>
-   <!-- Replace the fake hardware section with this: -->
+   <!-- OnRobot 2FG7 Gripper - Supports both simulation and real hardware -->
+   <xacro:if value="$(arg use_fake_hardware)">
+   <!-- Simulation mode -->
+   <ros2_control name="onrobot_2fg7_gripper" type="system">
+      <hardware>
+         <plugin>mock_components/GenericSystem</plugin>
+         <param name="fake_sensor_commands">$(arg fake_sensor_commands)</param>
+      </hardware>
+      <joint name="left_finger_joint">
+         <command_interface name="position"/>
+         <state_interface name="position"/>
+         <state_interface name="velocity"/>
+      </joint>
+      <joint name="right_finger_joint">
+         <command_interface name="position"/>
+         <state_interface name="position"/>
+         <state_interface name="velocity"/>
+      </joint>
+   </ros2_control>
+   </xacro:if>
    <xacro:unless value="$(arg use_fake_hardware)">
+   <!-- Real hardware mode -->
    <ros2_control name="onrobot_2fg7_gripper" type="system">
       <hardware>
@@ -213,22 +233,3 @@
    </ros2_control>
    </xacro:unless>
-   <xacro:if value="$(arg use_fake_hardware)">
-   <!-- Keep the fake hardware for simulation -->
-   <ros2_control name="onrobot_2fg7_gripper" type="system">
-      <hardware>
-         <plugin>mock_components/GenericSystem</plugin>
-         <param name="fake_sensor_commands">$(arg fake_sensor_commands)</param>
-      </hardware>
-      <joint name="left_finger_joint">
-         <command_interface name="position"/>
-         <state_interface name="position"/>
-         <state_interface name="velocity"/>
-      </joint>
-      <joint name="right_finger_joint">
-         <command_interface name="position"/>
-         <state_interface name="position"/>
-         <state_interface name="velocity"/>
-      </joint>
-   </ros2_control>
-</xacro:if>
 </robot>

Commit message: Third Approach

File: drims2_description/urdf/ur5e_2fg7/ur5e_2fg7_cell.urdf.xacro (robot description, xacro)
@@ -210,25 +210,25 @@
    <!-- Real hardware mode -->
    <ros2_control name="onrobot_2fg7_gripper" type="system">
-      <hardware>
-         <plugin>onrobot_driver/OnRobotGripperHardwareInterface</plugin>
-         <param name="ip_address">192.168.1.1</param>
-         <param name="port">502</param>
-         <param name="gripper_type">2FG7</param>
-         <param name="max_width">0.085</param>
-         <param name="min_width">0.0</param>
-         <param name="max_force">100.0</param>
-      </hardware>
-      <joint name="left_finger_joint">
-         <command_interface name="position"/>
-         <state_interface name="position"/>
-         <state_interface name="velocity"/>
-         <state_interface name="effort"/>
-      </joint>
-      <joint name="right_finger_joint">
-         <command_interface name="position"/>
-         <state_interface name="position"/>
-         <state_interface name="velocity"/>
-         <state_interface name="effort"/>
-      </joint>
+   <hardware>
+      <plugin>onrobot_driver/OnRobotGripperHardwareInterface</plugin>
+      <param name="ip_address">192.168.1.1</param>
+      <param name="port">502</param>
+      <param name="gripper_type">2FG7</param>
+      <param name="max_width">0.085</param>
+      <param name="min_width">0.0</param>
+      <param name="max_force">100.0</param>
+   </hardware>
+   <joint name="left_finger_joint">
+      <command_interface name="position"/>
+      <state_interface name="position"/>
+      <state_interface name="velocity"/>
+      <state_interface name="effort"/>
+   </joint>
+   <joint name="right_finger_joint">
+      <command_interface name="position"/>
+      <state_interface name="position"/>
+      <state_interface name="velocity"/>
+      <state_interface name="effort"/>
+   </joint>
    </ros2_control>
    </xacro:unless>

Commit message: 6 - oct - integrating onrobot driver

File: drims2_description/urdf/ur5e_2fg7/ur5e_2fg7_cell.urdf.xacro (robot description, xacro)
@@ -188,7 +188,6 @@
       <origin xyz="0 0 0.15" rpy="0 0 0"/>
    </joint>
-   <!-- OnRobot 2FG7 Gripper - Supports both simulation and real hardware -->
-   <xacro:if value="$(arg use_fake_hardware)">
-   <!-- Simulation mode -->
+   <!-- OnRobot 2FG7 Gripper - SIMPLIFIED: Only simulation mode in hardware interface -->
+   <!-- Real hardware communication is handled by the separate onrobot_driver_node -->
    <ros2_control name="onrobot_2fg7_gripper" type="system">
       <hardware>
@@ -207,30 +206,3 @@
       </joint>
    </ros2_control>
-   </xacro:if>
-   <xacro:unless value="$(arg use_fake_hardware)">
-   <!-- Real hardware mode -->
-   <ros2_control name="onrobot_2fg7_gripper" type="system">
-   <hardware>
-      <plugin>onrobot_driver/OnRobotGripperHardwareInterface</plugin>
-      <param name="ip_address">192.168.1.1</param>
-      <param name="port">502</param>
-      <param name="gripper_type">2FG7</param>
-      <param name="max_width">0.085</param>
-      <param name="min_width">0.0</param>
-      <param name="max_force">100.0</param>
-   </hardware>
-   <joint name="left_finger_joint">
-      <command_interface name="position"/>
-      <state_interface name="position"/>
-      <state_interface name="velocity"/>
-      <state_interface name="effort"/>
-   </joint>
-   <joint name="right_finger_joint">
-      <command_interface name="position"/>
-      <state_interface name="position"/>
-      <state_interface name="velocity"/>
-      <state_interface name="effort"/>
-   </joint>
-   </ros2_control>
-   </xacro:unless>
 </robot>

Commit message: Joint name mismatch standardization

File: drims2_description/urdf/ur5e_2fg7/ur5e_2fg7_cell.urdf.xacro (robot description, xacro)
@@ -202,16 +202,16 @@
          <!-- FIX: Correct initial positions for gripper joints -->
          <param name="state_initial_values">
-            left_finger_joint/position: 0.010  # Start at mid-position (55mm opening)
-            left_finger_joint/velocity: 0.0
-            right_finger_joint/position: -0.010  # Mirror of left finger
-            right_finger_joint/velocity: 0.0
+            2fg7_left_finger_joint/position: 0.010  # Start at mid-position (55mm opening)
+            2fg7_left_finger_joint/velocity: 0.0
+            2fg7_right_finger_joint/position: -0.010  # Mirror of left finger
+            2fg7_right_finger_joint/velocity: 0.0
          </param>
       </hardware>
-      <joint name="left_finger_joint">
+      <joint name="2fg7_left_finger_joint">
          <command_interface name="position"/>
          <state_interface name="position"/>
          <state_interface name="velocity"/>
       </joint>
-      <joint name="right_finger_joint">
+      <joint name="2fg7_right_finger_joint">
          <command_interface name="position"/>
          <state_interface name="position"/>

Commit message: Joint name mismatch standardization

File: drims2_description/urdf/ur5e_2fg7/ur5e_2fg7_cell.urdf.xacro (robot description, xacro)
@@ -202,16 +202,16 @@
          <!-- FIX: Correct initial positions for gripper joints -->
          <param name="state_initial_values">
-            2fg7_left_finger_joint/position: 0.010  # Start at mid-position (55mm opening)
-            2fg7_left_finger_joint/velocity: 0.0
-            2fg7_right_finger_joint/position: -0.010  # Mirror of left finger
-            2fg7_right_finger_joint/velocity: 0.0
+            left_finger_joint/position: 0.010  # Start at mid-position (55mm opening)
+            left_finger_joint/velocity: 0.0
+            right_finger_joint/position: -0.010  # Mirror of left finger
+            right_finger_joint/velocity: 0.0
          </param>
       </hardware>
-      <joint name="2fg7_left_finger_joint">
+      <joint name="left_finger_joint">
          <command_interface name="position"/>
          <state_interface name="position"/>
          <state_interface name="velocity"/>
       </joint>
-      <joint name="2fg7_right_finger_joint">
+      <joint name="right_finger_joint">
          <command_interface name="position"/>
          <state_interface name="position"/>

Commit message: modifying tables

File: drims2_description/urdf/ur5e_2fg7/ur5e_2fg7_cell.urdf.xacro (robot description, xacro)
@@ -41,7 +41,7 @@
    <link name="world"/>
    <xacro:property name="table_length" value="1.2"/>
-   <xacro:property name="table_width" value="0.6"/>
+   <xacro:property name="table_width" value="0.7"/>
    <xacro:property name="table_height" value="0.75"/>
-   <xacro:property name="table_thickness" value="0.05"/>
+   <xacro:property name="table_thickness" value="0.063"/>
    <xacro:property name="leg_width" value="0.05"/>
    <link name="table_top">
@@ -51,6 +51,6 @@
          </geometry>
          <origin xyz="0 0 -${table_thickness/2}" rpy="0 0 0"/>
-         <material name="brown">
-            <color rgba="0.4 0.2 0 1"/>
+         <material name="white">
+            <color rgba="1 1 1 1"/>
          </material>
       </visual>
@@ -77,6 +77,6 @@
             </geometry>
             <origin xyz="0 0 ${z / 2}" rpy="0 0 0"/>
-            <material name="black">
-               <color rgba="0.1 0.1 0.1 1"/>
+            <material name="gray">
+               <color rgba="0.53 0.53 0.53 1"/>
             </material>
          </visual>
@@ -126,12 +126,12 @@
    </xacro:macro>
    <xacro:safety_barrier name="barrier_back"
-   xyz="${-table_length/2 - 0.3} 0 0.3"
-   size="0.01 ${table_width} 0.8"/>
+   xyz="${-table_width/2 - 0.4} 0 0.3"
+   size="0.01 ${table_length} 0.8"/>
    <xacro:safety_barrier name="barrier_left"
-   xyz="0 ${-table_width/2 - 0.3} 0.3"
-   size="${table_length} 0.01 0.8"/>
+   xyz="0 ${-table_length/2 - 0.3} 0.3"
+   size="${table_width} 0.01 0.8"/>
    <xacro:safety_barrier name="barrier_right"
-   xyz="0 ${table_width/2 + 0.3} 0.3"
-   size="${table_length} 0.01 0.8"/>
+   xyz="0 ${table_length/2 + 0.4} 0.3"
+   size="${table_width} 0.01 0.8"/>
    <xacro:safety_barrier name="barrier_top"
    xyz="0 0 1.2"

Commit message: modifying environment - v1 - rotated white table

File: drims2_description/urdf/ur5e_2fg7/ur5e_2fg7_cell.urdf.xacro (robot description, xacro)
@@ -41,7 +41,7 @@
    <link name="world"/>
    <xacro:property name="table_length" value="1.2"/>
-   <xacro:property name="table_width" value="0.6"/>
+   <xacro:property name="table_width" value="0.7"/>
    <xacro:property name="table_height" value="0.75"/>
-   <xacro:property name="table_thickness" value="0.05"/>
+   <xacro:property name="table_thickness" value="0.063"/>
    <xacro:property name="leg_width" value="0.05"/>
    <link name="table_top">
@@ -51,6 +51,6 @@
          </geometry>
          <origin xyz="0 0 -${table_thickness/2}" rpy="0 0 0"/>
-         <material name="brown">
-            <color rgba="0.4 0.2 0 1"/>
+         <material name="white">
+            <color rgba="1 1 1 1"/>
          </material>
       </visual>
@@ -77,6 +77,6 @@
             </geometry>
             <origin xyz="0 0 ${z / 2}" rpy="0 0 0"/>
-            <material name="black">
-               <color rgba="0.1 0.1 0.1 1"/>
+            <material name="gray">
+               <color rgba="0.53 0.53 0.53 1"/>
             </material>
          </visual>
@@ -126,12 +126,12 @@
    </xacro:macro>
    <xacro:safety_barrier name="barrier_back"
+   xyz="0 ${-table_length/2 + 0.4} 0.3"
+   size="${table_length} 0.01 0.8"/>
+   <xacro:safety_barrier name="barrier_left"
    xyz="${-table_length/2 - 0.3} 0 0.3"
    size="0.01 ${table_width} 0.8"/>
-   <xacro:safety_barrier name="barrier_left"
-   xyz="0 ${-table_width/2 - 0.3} 0.3"
-   size="${table_length} 0.01 0.8"/>
    <xacro:safety_barrier name="barrier_right"
-   xyz="0 ${table_width/2 + 0.3} 0.3"
-   size="${table_length} 0.01 0.8"/>
+   xyz="-0.4 0 0.3"
+   size="0.01 ${table_width} 0.8"/>
    <xacro:safety_barrier name="barrier_top"
    xyz="0 0 1.2"
@@ -175,5 +175,5 @@
       trajectory_port="$(arg trajectory_port)"
       >
-      <origin xyz="${-table_length/2.0 + 0.1} 0 0" rpy="0 0 0"/>
+      <origin xyz="0 ${-table_width/2.0 + 0.175} 0" rpy="0 0 0"/>
    </xacro:ur_robot>
    <!-- GRIPPER ATTACHMENT -->

Commit message: modifying environment - v2 - including conveyor belt

File: drims2_description/urdf/ur5e_2fg7/ur5e_2fg7_cell.urdf.xacro (robot description, xacro)
@@ -40,4 +40,5 @@
    <xacro:property name="initial_positions_file" default="$(arg initial_positions_file)"/>
    <link name="world"/>
+   <!-- TABLE PROPERTIES -->
    <xacro:property name="table_length" value="1.2"/>
    <xacro:property name="table_width" value="0.7"/>
@@ -45,4 +46,5 @@
    <xacro:property name="table_thickness" value="0.063"/>
    <xacro:property name="leg_width" value="0.05"/>
+   <!-- TABLE DEFINITION -->
    <link name="table_top">
       <visual>
@@ -65,8 +67,9 @@
       </collision>
    </link>
+   <!-- Table rotated 90 degrees (1.5708 radians) around Z-axis -->
    <joint name="world_to_table" type="fixed">
       <parent link="world"/>
       <child link="table_top"/>
-      <origin xyz="0 0 ${table_height}" rpy="0 0 0"/>
+      <origin xyz="0 0 ${table_height}" rpy="0 0 1.5708"/>
    </joint>
    <xacro:macro name="table_leg" params="name x y z">
@@ -94,5 +97,6 @@
          <parent link="world"/>
          <child link="${name}"/>
-         <origin xyz="${x} ${y} 0" rpy="0 0 0"/>
+         <!-- Leg positions also rotated 90 degrees -->
+         <origin xyz="${-y} ${x} 0" rpy="0 0 1.5708"/>
          </joint>
    </xacro:macro>
@@ -125,16 +129,131 @@
    </joint>
    </xacro:macro>
+   <!-- Safety barriers positions adjusted for 90-degree rotation -->
    <xacro:safety_barrier name="barrier_back"
-   xyz="0 ${-table_length/2 + 0.4} 0.3"
-   size="${table_length} 0.01 0.8"/>
+   xyz="${-table_width/2 - 0.3} 0 0.3"
+   size="0.01 ${table_length} 0.8"/>
    <xacro:safety_barrier name="barrier_left"
-   xyz="${-table_length/2 - 0.3} 0 0.3"
-   size="0.01 ${table_width} 0.8"/>
+   xyz="0 ${-table_length/2 - 0.3} 0.3"
+   size="${table_width} 0.01 0.8"/>
    <xacro:safety_barrier name="barrier_right"
-   xyz="-0.4 0 0.3"
-   size="0.01 ${table_width} 0.8"/>
+   xyz="0 ${table_length/2 + 0.3} 0.3"
+   size="${table_width} 0.01 0.8"/>
    <xacro:safety_barrier name="barrier_top"
    xyz="0 0 1.2"
-   size="${table_length} ${table_width} 0.01"/>
+   size="${table_width} ${table_length} 0.01"/>
+   <!-- CONVEYOR BELT PROPERTIES -->
+   <xacro:property name="conveyor_length" value="1.5"/>
+   <xacro:property name="conveyor_width" value="0.4"/>
+   <xacro:property name="conveyor_height" value="0.85"/>
+   <xacro:property name="conveyor_thickness" value="0.02"/>
+   <xacro:property name="conveyor_leg_width" value="0.04"/>
+   <!-- CONVEYOR BELT DEFINITION -->
+   <!-- Conveyor belt surface -->
+   <link name="conveyor_belt">
+      <visual>
+         <geometry>
+            <box size="${conveyor_length} ${conveyor_width} ${conveyor_thickness}"/>
+         </geometry>
+         <origin xyz="0 0 -${conveyor_thickness/2}" rpy="0 0 0"/>
+         <material name="dark_green_rubber">
+            <color rgba="0 0.43 0 1"/>
+         </material>
+      </visual>
+      <collision>
+         <geometry>
+            <box size="${conveyor_length} ${conveyor_width} ${conveyor_thickness}"/>
+         </geometry>
+         <origin xyz="0 0 -${conveyor_thickness/2}" rpy="0 0 0"/>
+      </collision>
+   </link>
+   <!-- Conveyor frame -->
+   <link name="conveyor_frame">
+      <visual>
+         <geometry>
+            <box size="${conveyor_length} ${conveyor_width + 0.1} 0.05"/>
+         </geometry>
+         <origin xyz="0 0 -0.025" rpy="0 0 0"/>
+         <material name="aluminum">
+            <color rgba="0.8 0.8 0.8 1"/>
+         </material>
+      </visual>
+      <collision>
+         <geometry>
+            <box size="${conveyor_length} ${conveyor_width + 0.1} 0.05"/>
+         </geometry>
+         <origin xyz="0 0 -0.025" rpy="0 0 0"/>
+      </collision>
+   </link>
+   <!-- Joint connecting conveyor belt to frame -->
+   <joint name="conveyor_belt_to_frame" type="fixed">
+      <parent link="conveyor_frame"/>
+      <child link="conveyor_belt"/>
+      <origin xyz="0 0 ${conveyor_thickness/2 + 0.025}" rpy="0 0 0"/>
+   </joint>
+   <!-- Conveyor positioned in FRONT of the table and rotated 90 degrees -->
+   <joint name="world_to_conveyor" type="fixed">
+      <parent link="world"/>
+      <child link="conveyor_frame"/>
+      <origin xyz="${table_width/2 + conveyor_width/2 + 0.05} 0 ${conveyor_height}" rpy="0 0 1.5708"/>
+   </joint>
+   <!-- Conveyor legs -->
+   <xacro:macro name="conveyor_leg" params="name x y z">
+      <link name="${name}">
+         <visual>
+            <geometry>
+               <box size="${conveyor_leg_width} ${conveyor_leg_width} ${z}"/>
+            </geometry>
+            <origin xyz="0 0 ${z / 2}" rpy="0 0 0"/>
+            <material name="steel">
+               <color rgba="0.5 0.5 0.5 1"/>
+            </material>
+         </visual>
+         <collision>
+            <geometry>
+               <box size="${conveyor_leg_width} ${conveyor_leg_width} ${z}"/>
+            </geometry>
+            <origin xyz="0 0 ${z / 2}" rpy="0 0 0"/>
+         </collision>
+      </link>
+      <joint name="joint_${name}" type="fixed">
+         <parent link="world"/>
+         <child link="${name}"/>
+         <!-- Conveyor leg positions also rotated 90 degrees -->
+         <origin xyz="${-y} ${x} 0" rpy="0 0 1.5708"/>
+      </joint>
+   </xacro:macro>
+   <!-- FIXED: Conveyor legs positioned at the correct corners for rotated conveyor -->
+   <!-- Since conveyor is rotated 90 degrees, we need to swap length/width in positioning -->
+   <xacro:conveyor_leg name="conveyor_leg_1" x="${-conveyor_length / 2 + conveyor_leg_width / 2}" y="${-(table_width/2 + conveyor_width/2 + 0.05 + conveyor_width / 2 - conveyor_leg_width / 2)}" z="${conveyor_height}"/>
+   <xacro:conveyor_leg name="conveyor_leg_2" x="${-conveyor_length / 2 + conveyor_leg_width / 2}" y="${-(table_width/2 + conveyor_width/2 + 0.05 - conveyor_width / 2 + conveyor_leg_width / 2)}" z="${conveyor_height}"/>
+   <xacro:conveyor_leg name="conveyor_leg_3" x="${conveyor_length / 2 - conveyor_leg_width / 2}" y="${-(table_width/2 + conveyor_width/2 + 0.05 + conveyor_width / 2 - conveyor_leg_width / 2)}" z="${conveyor_height}"/>
+   <xacro:conveyor_leg name="conveyor_leg_4" x="${conveyor_length / 2 - conveyor_leg_width / 2}" y="${-(table_width/2 + conveyor_width/2 + 0.05 - conveyor_width / 2 + conveyor_leg_width / 2)}" z="${conveyor_height}"/>
+   <!-- Optional: Conveyor end rollers -->
+   <!-- <xacro:macro name="conveyor_roller" params="name x_offset">
+      <link name="${name}">
+         <visual>
+            <geometry>
+               <cylinder length="${conveyor_width}" radius="0.05"/>
+            </geometry>
+            <origin xyz="0 0 0" rpy="0 1.5708 0"/>
+            <material name="rubber">
+               <color rgba="0.3 0.3 0.3 1"/>
+            </material>
+         </visual>
+         <collision>
+            <geometry>
+               <cylinder length="${conveyor_width}" radius="0.05"/>
+            </geometry>
+            <origin xyz="0 0 0" rpy="0 1.5708 0"/>
+         </collision>
+      </link>
+      <joint name="joint_${name}" type="fixed">
+         <parent link="conveyor_frame"/>
+         <child link="${name}"/>
+         <origin xyz="${x_offset} 0 0.025" rpy="0 0 0"/>
+      </joint>
+   </xacro:macro>
+   <xacro:conveyor_roller name="conveyor_roller_front" x_offset="${conveyor_length/2 - 0.05}"/>
+   <xacro:conveyor_roller name="conveyor_roller_back" x_offset="${-conveyor_length/2 + 0.05}"/> -->
    <!-- MAIN ROBOT - This includes the complete UR5e robot -->
    <xacro:ur_robot
@@ -175,5 +294,6 @@
       trajectory_port="$(arg trajectory_port)"
       >
-      <origin xyz="0 ${-table_width/2.0 + 0.175} 0" rpy="0 0 0"/>
+      <!-- Robot origin adjusted for the rotated table -->
+      <origin xyz="0.125 ${-table_width/2.0 + 0.225} 0" rpy="0 0 0"/>
    </xacro:ur_robot>
    <!-- GRIPPER ATTACHMENT -->
