Commit message: modifying environment - v2.1 - conveyor belt real values and legs positions

File: drims2_description/urdf/ur5e_2fg7/ur5e_2fg7_cell.urdf.xacro (robot description, xacro)
@@ -143,9 +143,11 @@
    size="${table_width} ${table_length} 0.01"/>
    <!-- CONVEYOR BELT PROPERTIES -->
-   <xacro:property name="conveyor_length" value="1.5"/>
-   <xacro:property name="conveyor_width" value="0.4"/>
-   <xacro:property name="conveyor_height" value="0.85"/>
-   <xacro:property name="conveyor_thickness" value="0.02"/>
-   <xacro:property name="conveyor_leg_width" value="0.04"/>
+   <xacro:property name="conveyor_length" value="2.05"/>
+   <xacro:property name="conveyor_width" value="0.8"/>
+   <xacro:property name="conveyor_height" value="0.8"/>
+   <xacro:property name="conveyor_thickness" value="0.002"/>
+   <xacro:property name="conveyor_leg_width" value="0.043"/>
+   <xacro:property name="conveyor_frame_width" value="0.84"/>
+   <xacro:property name="conveyor_frame_height" value="0.09"/>
    <!-- CONVEYOR BELT DEFINITION -->
    <!-- Conveyor belt surface -->
@@ -171,16 +173,16 @@
       <visual>
          <geometry>
-            <box size="${conveyor_length} ${conveyor_width + 0.1} 0.05"/>
-         </geometry>
-         <origin xyz="0 0 -0.025" rpy="0 0 0"/>
-         <material name="aluminum">
-            <color rgba="0.8 0.8 0.8 1"/>
+            <box size="${conveyor_length} ${conveyor_frame_width} ${conveyor_frame_height}"/>
+         </geometry>
+         <origin xyz="0 0 ${-conveyor_frame_height}" rpy="0 0 0"/>
+         <material name="gray_steel">
+            <color rgba="0.5 0.5 0.5 1"/>
          </material>
       </visual>
       <collision>
          <geometry>
-            <box size="${conveyor_length} ${conveyor_width + 0.1} 0.05"/>
-         </geometry>
-         <origin xyz="0 0 -0.025" rpy="0 0 0"/>
+            <box size="${conveyor_length} ${conveyor_frame_width} ${conveyor_frame_height}"/>
+         </geometry>
+         <origin xyz="0 0 ${-conveyor_frame_height}" rpy="0 0 0"/>
       </collision>
    </link>
@@ -195,5 +197,5 @@
       <parent link="world"/>
       <child link="conveyor_frame"/>
-      <origin xyz="${table_width/2 + conveyor_width/2 + 0.05} 0 ${conveyor_height}" rpy="0 0 1.5708"/>
+      <origin xyz="${table_width/2 + conveyor_width/2 + 0.115} 0 ${conveyor_height}" rpy="0 0 1.5708"/>
    </joint>
    <!-- Conveyor legs -->
@@ -225,8 +227,8 @@
    <!-- FIXED: Conveyor legs positioned at the correct corners for rotated conveyor -->
    <!-- Since conveyor is rotated 90 degrees, we need to swap length/width in positioning -->
-   <xacro:conveyor_leg name="conveyor_leg_1" x="${-conveyor_length / 2 + conveyor_leg_width / 2}" y="${-(table_width/2 + conveyor_width/2 + 0.05 + conveyor_width / 2 - conveyor_leg_width / 2)}" z="${conveyor_height}"/>
-   <xacro:conveyor_leg name="conveyor_leg_2" x="${-conveyor_length / 2 + conveyor_leg_width / 2}" y="${-(table_width/2 + conveyor_width/2 + 0.05 - conveyor_width / 2 + conveyor_leg_width / 2)}" z="${conveyor_height}"/>
-   <xacro:conveyor_leg name="conveyor_leg_3" x="${conveyor_length / 2 - conveyor_leg_width / 2}" y="${-(table_width/2 + conveyor_width/2 + 0.05 + conveyor_width / 2 - conveyor_leg_width / 2)}" z="${conveyor_height}"/>
-   <xacro:conveyor_leg name="conveyor_leg_4" x="${conveyor_length / 2 - conveyor_leg_width / 2}" y="${-(table_width/2 + conveyor_width/2 + 0.05 - conveyor_width / 2 + conveyor_leg_width / 2)}" z="${conveyor_height}"/>
+   <xacro:conveyor_leg name="conveyor_leg_1" x="${-conveyor_length / 2 + conveyor_leg_width / 2}" y="${-(table_width/2 + conveyor_width - 3 * conveyor_leg_width / 2)}" z="${conveyor_height - conveyor_frame_height}"/>
+   <xacro:conveyor_leg name="conveyor_leg_2" x="${-conveyor_length / 2 + conveyor_leg_width / 2}" y="${-(table_width/2 - conveyor_leg_width / 2)}" z="${conveyor_height - conveyor_frame_height}"/>
+   <xacro:conveyor_leg name="conveyor_leg_3" x="${conveyor_length / 2 - conveyor_leg_width / 2}" y="${-(table_width/2 + conveyor_width - 3 * conveyor_leg_width / 2)}" z="${conveyor_height - conveyor_frame_height}"/>
+   <xacro:conveyor_leg name="conveyor_leg_4" x="${conveyor_length / 2 - conveyor_leg_width / 2}" y="${-(table_width/2 - conveyor_leg_width / 2)}" z="${conveyor_height - conveyor_frame_height}"/>
    <!-- Optional: Conveyor end rollers -->
    <!-- <xacro:macro name="conveyor_roller" params="name x_offset">

Commit message: modifying environment - v3 - second table inclusion

File: drims2_description/urdf/ur5e_2fg7/ur5e_2fg7_cell.urdf.xacro (robot description, xacro)
@@ -46,5 +46,5 @@
    <xacro:property name="table_thickness" value="0.063"/>
    <xacro:property name="leg_width" value="0.05"/>
-   <!-- TABLE DEFINITION -->
+   <!-- FIRST TABLE DEFINITION -->
    <link name="table_top">
       <visual>
@@ -67,5 +67,5 @@
       </collision>
    </link>
-   <!-- Table rotated 90 degrees (1.5708 radians) around Z-axis -->
+   <!-- First table rotated 90 degrees (1.5708 radians) around Z-axis -->
    <joint name="world_to_table" type="fixed">
       <parent link="world"/>
@@ -142,4 +142,49 @@
    xyz="0 0 1.2"
    size="${table_width} ${table_length} 0.01"/>
+   <!-- SECOND TABLE DEFINITION (identical to first table but positioned on the other side) -->
+   <link name="table_top_2">
+      <visual>
+         <geometry>
+            <box size="${table_length} ${table_width} ${table_thickness}"/>
+         </geometry>
+         <origin xyz="0 0 -${table_thickness/2}" rpy="0 0 0"/>
+         <material name="white">
+            <color rgba="1 1 1 1"/>
+         </material>
+      </visual>
+      <collision>
+         <geometry>
+            <box size="${table_length} ${table_width} ${table_thickness}"/>
+         </geometry>
+         <origin xyz="0 0 -${table_thickness/2}" rpy="0 0 0"/>
+         <material name="brown">
+            <color rgba="0.4 0.2 0 1"/>
+         </material>
+      </collision>
+   </link>
+   <!-- Second table rotated 90 degrees and positioned on the other side of the conveyor -->
+   <joint name="world_to_table_2" type="fixed">
+      <parent link="world"/>
+      <child link="table_top_2"/>
+      <origin xyz="${conveyor_width + 2*table_width + 0.4} 0 ${table_height}" rpy="0 0 1.5708"/>
+   </joint>
+   <!-- Second table legs -->
+   <xacro:table_leg name="leg_1_table2" x="${table_length / 2 - leg_width / 2 + conveyor_width + 2*table_width + 0.4}" y="${table_width / 2 - leg_width / 2}" z="${table_height - table_thickness}"/>
+   <xacro:table_leg name="leg_2_table2" x="${-table_length / 2 + leg_width / 2 + conveyor_width + 2*table_width + 0.4}" y="${table_width / 2 - leg_width / 2}" z="${table_height - table_thickness}"/>
+   <xacro:table_leg name="leg_3_table2" x="${table_length / 2 - leg_width / 2 + conveyor_width + 2*table_width + 0.4}" y="${-table_width / 2 + leg_width / 2}" z="${table_height - table_thickness}"/>
+   <xacro:table_leg name="leg_4_table2" x="${-table_length / 2 + leg_width / 2 + conveyor_width + 2*table_width + 0.4}" y="${-table_width / 2 + leg_width / 2}" z="${table_height - table_thickness}"/>
+   <!-- Second table safety barriers -->
+   <xacro:safety_barrier name="barrier_back_table2"
+   xyz="${-table_width/2 - 0.3} 0 0.3"
+   size="0.01 ${table_length} 0.8"/>
+   <xacro:safety_barrier name="barrier_left_table2"
+   xyz="0 ${-table_length/2 - 0.3} 0.3"
+   size="${table_width} 0.01 0.8"/>
+   <xacro:safety_barrier name="barrier_right_table2"
+   xyz="0 ${table_length/2 + 0.3} 0.3"
+   size="${table_width} 0.01 0.8"/>
+   <xacro:safety_barrier name="barrier_top_table2"
+   xyz="0 0 1.2"
+   size="${table_width} ${table_length} 0.01"/>
    <!-- CONVEYOR BELT PROPERTIES -->
    <xacro:property name="conveyor_length" value="2.05"/>
@@ -193,9 +238,9 @@
       <origin xyz="0 0 ${conveyor_thickness/2 + 0.025}" rpy="0 0 0"/>
    </joint>
-   <!-- Conveyor positioned in FRONT of the table and rotated 90 degrees -->
+   <!-- Conveyor positioned between both tables -->
    <joint name="world_to_conveyor" type="fixed">
       <parent link="world"/>
       <child link="conveyor_frame"/>
-      <origin xyz="${table_width/2 + conveyor_width/2 + 0.115} 0 ${conveyor_height}" rpy="0 0 1.5708"/>
+      <origin xyz="${table_width + conveyor_width/2 + 0.2} 0 ${conveyor_height}" rpy="0 0 1.5708"/>
    </joint>
    <!-- Conveyor legs -->
@@ -225,37 +270,9 @@
       </joint>
    </xacro:macro>
-   <!-- FIXED: Conveyor legs positioned at the correct corners for rotated conveyor -->
-   <!-- Since conveyor is rotated 90 degrees, we need to swap length/width in positioning -->
-   <xacro:conveyor_leg name="conveyor_leg_1" x="${-conveyor_length / 2 + conveyor_leg_width / 2}" y="${-(table_width/2 + conveyor_width - 3 * conveyor_leg_width / 2)}" z="${conveyor_height - conveyor_frame_height}"/>
-   <xacro:conveyor_leg name="conveyor_leg_2" x="${-conveyor_length / 2 + conveyor_leg_width / 2}" y="${-(table_width/2 - conveyor_leg_width / 2)}" z="${conveyor_height - conveyor_frame_height}"/>
-   <xacro:conveyor_leg name="conveyor_leg_3" x="${conveyor_length / 2 - conveyor_leg_width / 2}" y="${-(table_width/2 + conveyor_width - 3 * conveyor_leg_width / 2)}" z="${conveyor_height - conveyor_frame_height}"/>
-   <xacro:conveyor_leg name="conveyor_leg_4" x="${conveyor_length / 2 - conveyor_leg_width / 2}" y="${-(table_width/2 - conveyor_leg_width / 2)}" z="${conveyor_height - conveyor_frame_height}"/>
-   <!-- Optional: Conveyor end rollers -->
-   <!-- <xacro:macro name="conveyor_roller" params="name x_offset">
-      <link name="${name}">
-         <visual>
-            <geometry>
-               <cylinder length="${conveyor_width}" radius="0.05"/>
-            </geometry>
-            <origin xyz="0 0 0" rpy="0 1.5708 0"/>
-            <material name="rubber">
-               <color rgba="0.3 0.3 0.3 1"/>
-            </material>
-         </visual>
-         <collision>
-            <geometry>
-               <cylinder length="${conveyor_width}" radius="0.05"/>
-            </geometry>
-            <origin xyz="0 0 0" rpy="0 1.5708 0"/>
-         </collision>
-      </link>
-      <joint name="joint_${name}" type="fixed">
-         <parent link="conveyor_frame"/>
-         <child link="${name}"/>
-         <origin xyz="${x_offset} 0 0.025" rpy="0 0 0"/>
-      </joint>
-   </xacro:macro>
-   <xacro:conveyor_roller name="conveyor_roller_front" x_offset="${conveyor_length/2 - 0.05}"/>
-   <xacro:conveyor_roller name="conveyor_roller_back" x_offset="${-conveyor_length/2 + 0.05}"/> -->
+   <!-- Conveyor legs positioned at the correct corners for rotated conveyor -->
+   <xacro:conveyor_leg name="conveyor_leg_1" x="${-conveyor_length / 2 + conveyor_leg_width / 2 + table_width + conveyor_width/2 + 0.2}" y="${-(table_width/2 + conveyor_width - 3 * conveyor_leg_width / 2)}" z="${conveyor_height - conveyor_frame_height}"/>
+   <xacro:conveyor_leg name="conveyor_leg_2" x="${-conveyor_length / 2 + conveyor_leg_width / 2 + table_width + conveyor_width/2 + 0.2}" y="${-(table_width/2 - conveyor_leg_width / 2)}" z="${conveyor_height - conveyor_frame_height}"/>
+   <xacro:conveyor_leg name="conveyor_leg_3" x="${conveyor_length / 2 - conveyor_leg_width / 2 + table_width + conveyor_width/2 + 0.2}" y="${-(table_width/2 + conveyor_width - 3 * conveyor_leg_width / 2)}" z="${conveyor_height - conveyor_frame_height}"/>
+   <xacro:conveyor_leg name="conveyor_leg_4" x="${conveyor_length / 2 - conveyor_leg_width / 2 + table_width + conveyor_width/2 + 0.2}" y="${-(table_width/2 - conveyor_leg_width / 2)}" z="${conveyor_height - conveyor_frame_height}"/>
    <!-- MAIN ROBOT - This includes the complete UR5e robot -->
    <xacro:ur_robot

Commit message: modifying environment - v4 - barrier fix + second table and conveyor belt fix + robot 180º rotated

File: drims2_description/urdf/ur5e_2fg7/ur5e_2fg7_cell.urdf.xacro (robot description, xacro)
@@ -129,62 +129,4 @@
    </joint>
    </xacro:macro>
-   <!-- Safety barriers positions adjusted for 90-degree rotation -->
-   <xacro:safety_barrier name="barrier_back"
-   xyz="${-table_width/2 - 0.3} 0 0.3"
-   size="0.01 ${table_length} 0.8"/>
-   <xacro:safety_barrier name="barrier_left"
-   xyz="0 ${-table_length/2 - 0.3} 0.3"
-   size="${table_width} 0.01 0.8"/>
-   <xacro:safety_barrier name="barrier_right"
-   xyz="0 ${table_length/2 + 0.3} 0.3"
-   size="${table_width} 0.01 0.8"/>
-   <xacro:safety_barrier name="barrier_top"
-   xyz="0 0 1.2"
-   size="${table_width} ${table_length} 0.01"/>
-   <!-- SECOND TABLE DEFINITION (identical to first table but positioned on the other side) -->
-   <link name="table_top_2">
-      <visual>
-         <geometry>
-            <box size="${table_length} ${table_width} ${table_thickness}"/>
-         </geometry>
-         <origin xyz="0 0 -${table_thickness/2}" rpy="0 0 0"/>
-         <material name="white">
-            <color rgba="1 1 1 1"/>
-         </material>
-      </visual>
-      <collision>
-         <geometry>
-            <box size="${table_length} ${table_width} ${table_thickness}"/>
-         </geometry>
-         <origin xyz="0 0 -${table_thickness/2}" rpy="0 0 0"/>
-         <material name="brown">
-            <color rgba="0.4 0.2 0 1"/>
-         </material>
-      </collision>
-   </link>
-   <!-- Second table rotated 90 degrees and positioned on the other side of the conveyor -->
-   <joint name="world_to_table_2" type="fixed">
-      <parent link="world"/>
-      <child link="table_top_2"/>
-      <origin xyz="${conveyor_width + 2*table_width + 0.4} 0 ${table_height}" rpy="0 0 1.5708"/>
-   </joint>
-   <!-- Second table legs -->
-   <xacro:table_leg name="leg_1_table2" x="${table_length / 2 - leg_width / 2 + conveyor_width + 2*table_width + 0.4}" y="${table_width / 2 - leg_width / 2}" z="${table_height - table_thickness}"/>
-   <xacro:table_leg name="leg_2_table2" x="${-table_length / 2 + leg_width / 2 + conveyor_width + 2*table_width + 0.4}" y="${table_width / 2 - leg_width / 2}" z="${table_height - table_thickness}"/>
-   <xacro:table_leg name="leg_3_table2" x="${table_length / 2 - leg_width / 2 + conveyor_width + 2*table_width + 0.4}" y="${-table_width / 2 + leg_width / 2}" z="${table_height - table_thickness}"/>
-   <xacro:table_leg name="leg_4_table2" x="${-table_length / 2 + leg_width / 2 + conveyor_width + 2*table_width + 0.4}" y="${-table_width / 2 + leg_width / 2}" z="${table_height - table_thickness}"/>
-   <!-- Second table safety barriers -->
-   <xacro:safety_barrier name="barrier_back_table2"
-   xyz="${-table_width/2 - 0.3} 0 0.3"
-   size="0.01 ${table_length} 0.8"/>
-   <xacro:safety_barrier name="barrier_left_table2"
-   xyz="0 ${-table_length/2 - 0.3} 0.3"
-   size="${table_width} 0.01 0.8"/>
-   <xacro:safety_barrier name="barrier_right_table2"
-   xyz="0 ${table_length/2 + 0.3} 0.3"
-   size="${table_width} 0.01 0.8"/>
-   <xacro:safety_barrier name="barrier_top_table2"
-   xyz="0 0 1.2"
-   size="${table_width} ${table_length} 0.01"/>
    <!-- CONVEYOR BELT PROPERTIES -->
    <xacro:property name="conveyor_length" value="2.05"/>
@@ -192,5 +134,5 @@
    <xacro:property name="conveyor_height" value="0.8"/>
    <xacro:property name="conveyor_thickness" value="0.002"/>
-   <xacro:property name="conveyor_leg_width" value="0.043"/>
+   <xacro:property name="conveyor_leg_width" value="0.045"/>
    <xacro:property name="conveyor_frame_width" value="0.84"/>
    <xacro:property name="conveyor_frame_height" value="0.09"/>
@@ -242,5 +184,5 @@
       <parent link="world"/>
       <child link="conveyor_frame"/>
-      <origin xyz="${table_width + conveyor_width/2 + 0.2} 0 ${conveyor_height}" rpy="0 0 1.5708"/>
+      <origin xyz="${table_width/2 + conveyor_width/2 + 0.08} ${0.4} ${conveyor_height}" rpy="0 0 1.5708"/>
    </joint>
    <!-- Conveyor legs -->
@@ -249,5 +191,5 @@
          <visual>
             <geometry>
-               <box size="${conveyor_leg_width} ${conveyor_leg_width} ${z}"/>
+               <box size="${2*conveyor_leg_width} ${conveyor_leg_width} ${z}"/>
             </geometry>
             <origin xyz="0 0 ${z / 2}" rpy="0 0 0"/>
@@ -258,5 +200,5 @@
          <collision>
             <geometry>
-               <box size="${conveyor_leg_width} ${conveyor_leg_width} ${z}"/>
+               <box size="${2*conveyor_leg_width} ${conveyor_leg_width} ${z}"/>
             </geometry>
             <origin xyz="0 0 ${z / 2}" rpy="0 0 0"/>
@@ -271,8 +213,69 @@
    </xacro:macro>
    <!-- Conveyor legs positioned at the correct corners for rotated conveyor -->
-   <xacro:conveyor_leg name="conveyor_leg_1" x="${-conveyor_length / 2 + conveyor_leg_width / 2 + table_width + conveyor_width/2 + 0.2}" y="${-(table_width/2 + conveyor_width - 3 * conveyor_leg_width / 2)}" z="${conveyor_height - conveyor_frame_height}"/>
-   <xacro:conveyor_leg name="conveyor_leg_2" x="${-conveyor_length / 2 + conveyor_leg_width / 2 + table_width + conveyor_width/2 + 0.2}" y="${-(table_width/2 - conveyor_leg_width / 2)}" z="${conveyor_height - conveyor_frame_height}"/>
-   <xacro:conveyor_leg name="conveyor_leg_3" x="${conveyor_length / 2 - conveyor_leg_width / 2 + table_width + conveyor_width/2 + 0.2}" y="${-(table_width/2 + conveyor_width - 3 * conveyor_leg_width / 2)}" z="${conveyor_height - conveyor_frame_height}"/>
-   <xacro:conveyor_leg name="conveyor_leg_4" x="${conveyor_length / 2 - conveyor_leg_width / 2 + table_width + conveyor_width/2 + 0.2}" y="${-(table_width/2 - conveyor_leg_width / 2)}" z="${conveyor_height - conveyor_frame_height}"/>
+   <xacro:conveyor_leg name="conveyor_leg_1" x="${-conveyor_length / 2 + conveyor_leg_width / 2  + 0.735}" y="${-(table_width/2 + conveyor_width + conveyor_leg_width + 0.08)}" z="${conveyor_height - conveyor_frame_height}"/>
+   <xacro:conveyor_leg name="conveyor_leg_2" x="${-conveyor_length / 2 + conveyor_leg_width / 2 + 0.735}" y="${-(table_width/2 - conveyor_leg_width + 0.08)}" z="${conveyor_height - conveyor_frame_height}"/>
+   <xacro:conveyor_leg name="conveyor_leg_3" x="${conveyor_length / 2 - conveyor_leg_width / 2 + 0.135}" y="${-(table_width/2 + conveyor_width + conveyor_leg_width + 0.08)}" z="${conveyor_height - conveyor_frame_height}"/>
+   <xacro:conveyor_leg name="conveyor_leg_4" x="${conveyor_length / 2 - conveyor_leg_width / 2 + 0.135}" y="${-(table_width/2 - conveyor_leg_width + 0.08)}" z="${conveyor_height - conveyor_frame_height}"/>
+   <!-- SECOND TABLE DEFINITION (identical to first table but positioned on the other side) -->
+   <link name="table_top_2">
+      <visual>
+         <geometry>
+            <box size="${table_length} ${table_width} ${table_thickness}"/>
+         </geometry>
+         <origin xyz="0 0 -${table_thickness/2}" rpy="0 0 0"/>
+         <material name="white">
+            <color rgba="1 1 1 1"/>
+         </material>
+      </visual>
+      <collision>
+         <geometry>
+            <box size="${table_length} ${table_width} ${table_thickness}"/>
+         </geometry>
+         <origin xyz="0 0 -${table_thickness/2}" rpy="0 0 0"/>
+         <material name="brown">
+            <color rgba="0.4 0.2 0 1"/>
+         </material>
+      </collision>
+   </link>
+   <!-- Second table rotated 90 degrees and positioned on the other side of the conveyor -->
+   <joint name="world_to_table_2" type="fixed">
+      <parent link="world"/>
+      <child link="table_top_2"/>
+      <origin xyz="${conveyor_width + table_width + 0.16} 0 ${table_height}" rpy="0 0 1.5708"/>
+   </joint>
+   <!-- Second table legs -->
+   <xacro:table_leg name="leg_back_right_table2" x="${table_length / 2 - leg_width / 2}" y="${-table_width/2 - conveyor_width - leg_width / 2  - 0.16}" z="${table_height - table_thickness}"/>
+   <xacro:table_leg name="leg_top_right_table2" x="${-table_length / 2 + leg_width / 2}" y="${-table_width/2 - conveyor_width - leg_width / 2 - 0.16}" z="${table_height - table_thickness}"/>
+   <xacro:table_leg name="leg_back_left_table2" x="${table_length / 2 - leg_width / 2}" y="${-3*table_width/2 - conveyor_width + leg_width / 2 - 0.16}" z="${table_height - table_thickness}"/>
+   <xacro:table_leg name="leg_top_left_table2" x="${-table_length / 2 + leg_width / 2}" y="${-3*table_width/2 - conveyor_width + leg_width / 2 - 0.16}" z="${table_height - table_thickness}"/>
+   <!-- Safety barriers positions adjusted for 90-degree rotation -->
+   <xacro:safety_barrier name="barrier_front"
+   xyz="0 ${- table_length/2 - conveyor_width + 0.16} 0.3"
+   size="${table_length} 0.01 0.8"/>
+   <xacro:safety_barrier name="barrier_back"
+   xyz="0 ${table_length/2 + 0.2} 0.3"
+   size="${table_length} 0.01 0.8"/>
+   <xacro:safety_barrier name="barrier_right"
+   xyz="${-table_length/2 + 0.15} 0 0.3"
+   size="0.01 ${table_width} 0.8"/>
+   <xacro:safety_barrier name="barrier_left"
+   xyz="${table_width/2 + 0.5} 0 0.3"
+   size="0.01 ${table_width} 0.8"/>
+   <xacro:safety_barrier name="barrier_top"
+   xyz="0 0 1.2"
+   size="${table_width} ${table_length} 0.01"/>
+   <!-- Second table safety barriers
+   <xacro:safety_barrier name="barrier_back_table2"
+   xyz="${-table_width/2 - 0.3} 0 0.3"
+   size="0.01 ${table_length} 0.8"/>
+   <xacro:safety_barrier name="barrier_left_table2"
+   xyz="0 ${-table_length/2 - 0.3} 0.3"
+   size="${table_width} 0.01 0.8"/>
+   <xacro:safety_barrier name="barrier_right_table2"
+   xyz="0 ${table_length/2 + 0.3} 0.3"
+   size="${table_width} 0.01 0.8"/>
+   <xacro:safety_barrier name="barrier_top_table2"
+   xyz="0 0 1.2"
+   size="${table_width} ${table_length} 0.01"/> -->
    <!-- MAIN ROBOT - This includes the complete UR5e robot -->
    <xacro:ur_robot
@@ -313,6 +316,6 @@
       trajectory_port="$(arg trajectory_port)"
       >
-      <!-- Robot origin adjusted for the rotated table -->
-      <origin xyz="0.125 ${-table_width/2.0 + 0.225} 0" rpy="0 0 0"/>
+      <!-- Robot origin rotated 180 degrees around Z-axis -->
+      <origin xyz="0.125 ${-table_width/2.0 + 0.225} 0" rpy="0 0 3.14159"/>
    </xacro:ur_robot>
    <!-- GRIPPER ATTACHMENT -->
